Commit message: Task 3 Fix: Add front_laser visual geometry, fix sensor plugin with gz-sim-sensors-system, update spawn.launch.py bridge to bidirectional

File: my_rb1_description/urdf/my_rb1_robot.urdf (robot description, URDF)
Before this commit: robot rb1_robot, 7 links, 6 joints
Links:
- link front_laser: mass None -> 0.1; geometry collision cylinder length=0.02 radius=0.01; visual cylinder length=0.02 radius=0.01
